File: atreus54.kicad_pcb (KiCad board)
At the start: 2 copper layers, 270.1 x 112.9 mm, 126 parts, among them SW1 SWITCH_PUSH, SW10 SWITCH_PUSH, SW11 SWITCH_PUSH, SW12 SWITCH_PUSH, SW13 SWITCH_PUSH, SW14 SWITCH_PUSH, SW15 SWITCH_PUSH, SW16 SWITCH_PUSH, SW17 SWITCH_PUSH, SW18 SWITCH_PUSH, SW19 SWITCH_PUSH, SW2 SWITCH_PUSH, SW20 SWITCH_PUSH, SW21 SWITCH_PUSH, SW22 SWITCH_PUSH, SW23 SWITCH_PUSH, SW24 SWITCH_PUSH, SW25 SWITCH_PUSH, SW26 SWITCH_PUSH, SW27 SWITCH_PUSH, SW28 SWITCH_PUSH, SW29 SWITCH_PUSH, SW3 SWITCH_PUSH, SW30 SWITCH_PUSH, SW31 SWITCH_PUSH, SW32 SWITCH_PUSH, SW33 SWITCH_PUSH, SW34 SWITCH_PUSH, SW35 SWITCH_PUSH, SW36 SWITCH_PUSH, SW37 SWITCH_PUSH, SW38 SWITCH_PUSH, SW39 SWITCH_PUSH, SW4 SWITCH_PUSH, SW40 SWITCH_PUSH, SW41 SWITCH_PUSH, SW42 SWITCH_PUSH, SW43 SWITCH_PUSH, SW44 SWITCH_PUSH, SW45 SWITCH_PUSH, SW46 SWITCH_PUSH, SW47 SWITCH_PUSH, SW48 SWITCH_PUSH, SW49 SWITCH_PUSH, SW5 SWITCH_PUSH, SW50 SWITCH_PUSH, SW51 SWITCH_PUSH, SW52 SWITCH_PUSH, SW53 SWITCH_PUSH, SW54 SWITCH_PUSH, SW55 SWITCH_PUSH, SW56 SWITCH_PUSH, SW57 SWITCH_PUSH, SW58 SWITCH_PUSH, SW59 SWITCH_PUSH, SW6 SWITCH_PUSH, SW60 SWITCH_PUSH, SW61 SWITCH_PUSH, SW62 SWITCH_PUSH, SW7 SWITCH_PUSH, SW8 SWITCH_PUSH, SW9 SWITCH_PUSH, U1 ARDUINO_PRO_MICRO

Commit message: remove wires
Routing:
- net /ROW4: track 353.1 -> 0.00 mm
- net /ROW0: track 328.4 -> 0.00 mm, vias 1 -> 0
- net /ROW3: track 316.2 -> 0.00 mm, vias 2 -> 0
- net /ROW1: track 300.5 -> 0.00 mm
- net /ROW2: track 297.3 -> 0.00 mm
- net /COL11: track 270.6 -> 0.00 mm, vias 6 -> 0
- net /COL12: track 264.8 -> 0.00 mm, vias 11 -> 0
- net /COL0: track 258.1 -> 0.00 mm, vias 4 -> 0
- net /COL10: track 252.7 -> 0.00 mm, vias 8 -> 0
- net /COL9: track 232.8 -> 0.00 mm, vias 2 -> 0
- net /COL1: track 225.2 -> 0.00 mm, vias 5 -> 0
- net /COL8: track 217.0 -> 0.00 mm, vias 4 -> 0
- net /COL2: track 206.5 -> 0.00 mm, vias 5 -> 0
- net /COL3: track 171.0 -> 0.00 mm, vias 6 -> 0
- net /COL4: track 162.8 -> 0.00 mm, vias 7 -> 0
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Other:
- net class Default removed
